File: Kicad/PCBstream/PCBstream.kicad_pcb (KiCad board)
At the start: 2 copper layers, 116.7 x 90.5 mm, 46 parts, among them SW2 SW_SPDT_312, U1 Nice_Nano_V2

Commit message: updated kicad files
Parts:
- added B+2: Jumper_3_Open, Connector_Wire:SolderWire-0.25sqmm_1x03_P4.2mm_D0.65mm_OD1.7mm, F.Cu at (63.7, 67.3)
- added GND2: Jumper_3_Open, Connector_Wire:SolderWire-0.25sqmm_1x03_P4.2mm_D0.65mm_OD1.7mm, F.Cu at (63.7, 70.2)
- B+1: renamed from B+; footprint Connector_Wire:SolderWire-0.5sqmm_1x01_D0.9mm_OD2.1mm -> ScottoKeebs_Scotto:TestPoint
- GND1: renamed from GND; footprint Connector_Wire:SolderWire-0.5sqmm_1x01_D0.9mm_OD2.1mm -> ScottoKeebs_Scotto:TestPoint
- moved GND1 15.8 mm to (70.0, 72.0)
- moved B+1 15.6 mm to (65.7, 72.0)
- moved D12 15.1 mm to (116.0, 107.8)
- moved D14 15.1 mm to (154.1, 107.8)
- moved D18 15.1 mm to (116.0, 126.8)
- moved D2 15.1 mm to (116.0, 69.7)
- moved D4 15.1 mm to (154.1, 69.7)
- moved D7 15.1 mm to (116.0, 88.7)
- moved D9 15.1 mm to (154.1, 88.7)
- moved H5 15.1 mm to (154.1, 75.4)
- moved H6 15.1 mm to (154.1, 94.5)
- moved S1 15.1 mm to (87.4, 70.6)
- moved S10 15.1 mm to (163.6, 89.7)
- moved S11 15.1 mm to (87.4, 108.7)
- moved S12 15.1 mm to (106.4, 104.0)
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Connections:
- GND1 pad 1: Net-(GND1-Pad1) -> JMP_GND
- SW2 pad 1: Net-(SW2-B) -> JMP_B
- U1 pad 1: unconnected-(U1-Pad1) -> B_LEFT
- U1 pad 2: unconnected-(U1-0-Pad2) -> GND_LEFT
- U1 pad 23: Net-(GND1-Pad1) -> GND_RIGHT
- U1 pad 24: Net-(SW2-B) -> B_RIGHT
Routing:
- net JMP_B: track 0.00 -> 50.0 mm
- net Net-(SW2-B): track 47.7 -> 0.00 mm
- net Net-(GND1-Pad1): track 6.85 -> 0.00 mm
- net B_RIGHT: track 0.00 -> 4.57 mm
- net B_LEFT: track 0.00 -> 4.56 mm
- net GND_RIGHT: track 0.00 -> 4.42 mm
- net GND_LEFT: track 0.00 -> 4.41 mm
- net JMP_GND: track 0.00 -> 2.89 mm
- net Net-(SW2-A): track 43.0 -> 40.4 mm
