File: Kicad/PCBstream/PCBstream.kicad_sch (KiCad schematic)
At the start: 46 parts, among them SW2 SW_SPDT_312, U1 Nice_Nano_V2

Commit message: updated kicad files
Parts:
- added B+2, GND2: Jumper_3_Open, Connector_Wire:SolderWire-0.25sqmm_1x03_P4.2mm_D0.65mm_OD1.7mm, symbol Jumper:Jumper_3_Open
- B+1, GND1: footprint Connector_Wire:SolderWire-0.5sqmm_1x01_D0.9mm_OD2.1mm -> ScottoKeebs_Scotto:TestPoint
Connections:
- net GND_RIGHT: now reaches U1.23 (GND)
- net GND_RIGHT: now also GND2.3 (B); no longer GND1.1
- net B_LEFT: now reaches U1.1
- net B_LEFT: now also B+2.1 (A)
- net GND_LEFT: now reaches U1.2 (0)
- net GND_LEFT: now also GND2.1 (A)
- net B_RIGHT: now reaches U1.24 (B+)
- net B_RIGHT: now also B+2.3 (B); no longer SW2.1 (B)
- new net JMP_B: B+2.2 (C), SW2.1 (B)
- new net JMP_GND: GND1.1, GND2.2 (C)
Other:
- moved on the sheet: B+1, GND1, SW2
